Commit message: Fixed motion planning

File: urdf/blue_cylinder.urdf (robot description, URDF)
Before this commit: robot blue_cylinder, 1 links, 0 joints
Links:
- link base_link: mass 0.00001 -> 0.05; geometry collision cylinder length=0.025 radius=0.04; visual cylinder length=0.025 radius=0.04

File: urdf/red_cylinder.urdf (robot description, URDF)
Before this commit: robot red_cylinder, 1 links, 0 joints
Links:
- link base_link: mass 0.00001 -> 0.05; geometry collision cylinder length=0.025 radius=0.04; visual cylinder length=0.025 radius=0.04

File: urdf/yellow_cylinder.urdf (robot description, URDF)
Before this commit: robot yellow_cylinder, 1 links, 0 joints
Links:
- link base_link: mass 0.00001 -> 0.05; geometry collision cylinder length=0.025 radius=0.04; visual cylinder length=0.025 radius=0.04

Commit message: Fixed velocity issue with cylinders that caused loss of grip

File: urdf/blue_cylinder.urdf (robot description, URDF)
Before this commit: robot blue_cylinder, 1 links, 0 joints
Links:
- link base_link: geometry collision cylinder length=0.025 radius=0.045; visual cylinder length=0.025 radius=0.045

File: urdf/red_cylinder.urdf (robot description, URDF)
Before this commit: robot red_cylinder, 1 links, 0 joints
Links:
- link base_link: geometry collision cylinder length=0.025 radius=0.045; visual cylinder length=0.025 radius=0.045

File: urdf/yellow_cylinder.urdf (robot description, URDF)
Before this commit: robot yellow_cylinder, 1 links, 0 joints
Links:
- link base_link: geometry collision cylinder length=0.025 radius=0.045; visual cylinder length=0.025 radius=0.045
